Commit message: rb2_description:: Updated elevator controller for gazebo. Wheels parameters changed

File: rb2_description/robots/rb2_std.urdf.xacro (robot description, xacro)
@@ -22,5 +22,5 @@
 	<!-- Wheel parameters -->
 	<xacro:property name="wheel_offset_x" value="0.0"/>    <!-- x,y,z in translation from base_link to the center of the wheel -->
-	<xacro:property name="wheel_offset_y" value="0.262"/>
+	<xacro:property name="wheel_offset_y" value="0.26"/>
 	<xacro:property name="wheel_offset_z" value="0.025"/>
 	<!-- Castor paramters -->

File: rb2_description/urdf/elevator/elevator.gazebo.xacro (robot description, xacro)
@@ -8,5 +8,5 @@
 			<kd value="1.0" />
 			<fdir1 value="1 0 0"/>
-			<material>Gazebo/Yellow</material>
+			<material>Gazebo/Grey</material>
 			<turnGravityOff>false</turnGravityOff>
 			<!--kp>500000.0</kp>

File: rb2_description/urdf/elevator/elevator.transmission.xacro (robot description, xacro)
@@ -3,14 +3,14 @@
 	<!-- Rubber wheel transmission -->
 	<xacro:macro name="elevator_transmission" params="prefix">
-	<!-- Transmission is important to link the joints and the controller (see rb1_control/config/rb1_control.yaml)-->
 		<transmission name="${prefix}_platform_trans">
 			<type>transmission_interface/SimpleTransmission</type>
 			<joint name="${prefix}_platform_joint">
 				<!-- for the gazebo plugin -->
-				<!--hardwareInterface>EffortJointInterface</hardwareInterface-->
+				<hardwareInterface>EffortJointInterface</hardwareInterface>
 				<!-- for ros control controller -->
-				<hardwareInterface>hardware_interface/PositionJointInterface</hardwareInterface>
+				<!--hardwareInterface>hardware_interface/PositionJointInterface</hardwareInterface-->
 			</joint>
 			<actuator name="${prefix}_platform_joint_motor">
+				<hardwareInterface>EffortJointInterface</hardwareInterface>
 				<mechanicalReduction>1</mechanicalReduction>
 				<motorTorqueConstant>20</motorTorqueConstant>

File: rb2_description/urdf/elevator/elevator.urdf.xacro (robot description, xacro)
@@ -7,4 +7,10 @@
 	<!-- name : name of the link: -->
 	<!-- hq: selects model in high quality (.dae) -->
+   <xacro:macro name="solid_cuboid_inertia" params="m h d w">
+    <inertia  ixx="${(m*(h*h+d*d))/12}" ixy = "0" ixz = "0"
+              iyy="${(m*(w*w+d*d))/12}" iyz = "0"
+              izz="${(m*(w*w+h*h))/12}"
+     />
+  </xacro:macro>
 	<!-- ELEVATOR PLATFORM -->
 	<joint name="${prefix}_platform_joint" type="prismatic">
@@ -38,7 +44,12 @@
 			</geometry>
 		</collision>
+		<inertial>
+			<mass value="0.005" />
+			<origin xyz="0 0 -0.27" />
+			<solid_cuboid_inertia m="0.005" h="0.05" d="0.05" w="0.05"/>
+		</inertial>
 	</link>
-	<!--xacro:elevator_transmission prefix="${prefix}" />
-	<xacro:elevator_gazebo prefix="${prefix}" /-->
+	<xacro:elevator_transmission prefix="${prefix}" />
+	<xacro:elevator_gazebo prefix="${prefix}" />
 	</xacro:macro>
 </robot>

File: rb2_description/urdf/wheels/omni_wheel.urdf.xacro (robot description, xacro)
@@ -3,7 +3,7 @@
   <xacro:property name="M_PI" value="3.1415926535897931" />
   <!-- Wheels -->
-  <xacro:property name="omni_wheel_radius" value="0.075" />
+  <xacro:property name="omni_wheel_radius" value="0.073" />
   <xacro:property name="omni_wheel_height" value="0.070" />
-  <xacro:property name="omni_wheel_mass" value="0.3" /> <!-- in kg-->
+  <xacro:property name="omni_wheel_mass" value="0.01" />
   <xacro:macro name="cylinder_inertia" params="m r h">
     <inertia  ixx="${m*(3*r*r+h*h)/12}" ixy = "0" ixz = "0"
@@ -28,5 +28,5 @@
           <origin xyz="0 0 0" rpy="0 0 0" />
           <geometry>
-				    <mesh filename="package://rb2_description/meshes/wheels/rb2_omni_wheel.dae" />
+				    <mesh filename="package://rb2_description/meshes/wheels/rb2_omni_wheel_fake.dae" />
           </geometry>
         </xacro:if>
@@ -41,7 +41,15 @@
       <collision>
       <origin xyz="0 0 0" rpy="${M_PI/2} 0 0" />
-       <geometry>
+      <geometry>
          <sphere radius="${omni_wheel_radius}"/>
-       </geometry>
+      </geometry>
+      <surface>
+        <friction>
+          <ode>
+            <mu>0.0001</mu>
+            <mu2>0.0001</mu2>
+          </ode>
+        </friction>
+			</surface>
       </collision>
       <inertial>

File: rb2_description/urdf/wheels/rubber_wheel.gazebo.xacro (robot description, xacro)
@@ -3,10 +3,10 @@
 	<xacro:macro name="rubber_wheel_gazebo" params="prefix">
 		<gazebo reference="${prefix}_wheel_link">
-			<mu1 value="5.0"/>
-			<mu2 value="0.5"/>
+			<mu1 value="1.0"/>
+			<mu2 value="1.0"/>
 			<kp value="10000000.0" />
 			<kd value="1.0" />
 			<fdir1 value="1 0 0"/>
-			<material>Gazebo/Yellow</material>
+			<material>Gazebo/Grey</material>
 			<turnGravityOff>false</turnGravityOff>
 			<!--kp>500000.0</kp>

File: rb2_description/urdf/wheels/rubber_wheel.urdf.xacro (robot description, xacro)
@@ -7,5 +7,5 @@
 	<xacro:property name="wheel_radius" value="0.110" />
 	<xacro:property name="wheel_height" value="0.07" />
-	<xacro:property name="wheel_mass" value="1.0" /> <!-- in kg-->
+	<xacro:property name="wheel_mass" value="0.3" /> <!-- in kg-->
 	<xacro:macro name="cylinder_inertia" params="m r h">
 		<inertia	ixx="${m*(3*r*r+h*h)/12}" ixy = "0" ixz = "0"
