Commit message: Fix elevator

File: rb2_description/urdf/elevator/elevator.gazebo.xacro (robot description, xacro)
@@ -5,5 +5,5 @@
 			<mu1 value="5.0"/>
 			<mu2 value="0.5"/>
-			<kp value="10000000.0" />
+			<kp value="Infinity" />
 			<kd value="1.0" />
 			<fdir1 value="1 0 0"/>

File: rb2_description/urdf/elevator/elevator.transmission.xacro (robot description, xacro)
@@ -7,10 +7,10 @@
 			<joint name="${prefix}_platform_joint">
 				<!-- for the gazebo plugin -->
-				<hardwareInterface>hardware_interface/EffortJointInterface</hardwareInterface>
+				<!--hardwareInterface>hardware_interface/EffortJointInterface</hardwareInterface-->
 				<!-- for ros control controller -->
-				<!--hardwareInterface>hardware_interface/PositionJointInterface</hardwareInterface-->
+				<hardwareInterface>hardware_interface/PositionJointInterface</hardwareInterface>
 			</joint>
 			<actuator name="${prefix}_platform_joint_motor">
-				<hardwareInterface>EffortJointInterface</hardwareInterface>
+				<hardwareInterface>PositionJointInterface</hardwareInterface>
 				<mechanicalReduction>1</mechanicalReduction>
 				<motorTorqueConstant>20</motorTorqueConstant>

File: rb2_description/urdf/elevator/elevator.urdf.xacro (robot description, xacro)
@@ -19,5 +19,6 @@
 			<child link="${prefix}_platform_link" />
 			<axis xyz="0 0 1"/>
-			<limit effort="1.0" lower="0.0" upper="0.05" velocity="0.5"/>
+			<limit effort="100.0" lower="0.0" upper="0.05" velocity="0.5"/>
+			<dynamics damping="0.7"/>
 	</joint>
 	<link name="${prefix}_platform_link">
@@ -45,7 +46,7 @@
 		</collision>
 		<inertial>
-			<mass value="0.005" />
+			<mass value="0.05" />
 			<origin xyz="0 0 -0.27" />
-			<solid_cuboid_inertia m="0.005" h="0.05" d="0.05" w="0.05"/>
+			<solid_cuboid_inertia m="0.05" h="0.05" d="0.05" w="0.05"/>
 		</inertial>
 	</link>
