Commit message: description: updating effort and transmission

File: rb2_description/urdf/elevator/elevator.transmission.xacro (robot description, xacro)
@@ -14,5 +14,4 @@
 				<hardwareInterface>EffortJointInterface</hardwareInterface>
 				<mechanicalReduction>1</mechanicalReduction>
-				<motorTorqueConstant>20</motorTorqueConstant>
 			</actuator>
 		</transmission>

File: rb2_description/urdf/elevator/elevator.urdf.xacro (robot description, xacro)
@@ -19,5 +19,5 @@
 			<child link="${prefix}_platform_link" />
 			<axis xyz="0 0 1"/>
-			<limit effort="1.0" lower="0.0" upper="0.05" velocity="0.5"/>
+			<limit effort="1000.0" lower="0.0" upper="0.05" velocity="0.01"/>
 	</joint>
 	<link name="${prefix}_platform_link">
@@ -39,8 +39,11 @@
 		</visual>
 		<collision>
-			<origin xyz="0 0 0" rpy="0 0 0 " />
+			<origin xyz="0 0 -0.0" rpy="0 0 0 " />
+			<!--geometry>
+				<box size="0.837 0.590 0.05" />
+			</geometry-->
 			<geometry>
-				<mesh filename="package://rb2_description/meshes/elevator/rb2_elevator.dae"/>
-			</geometry>
+					<mesh filename="package://rb2_description/meshes/elevator/rb2_elevator.dae"/>
+				</geometry>
 		</collision>
 		<inertial>
