Commit message: joint and link name changed. elevator upper limit updated

File: rb2_description/urdf/elevator/elevator.urdf.xacro (robot description, xacro)
@@ -8,12 +8,12 @@
 	<!-- hq: selects model in high quality (.dae) -->
 	<!-- ELEVATOR PLATFORM -->
-	<joint name="${prefix}_elevator_joint" type="prismatic">
+	<joint name="${prefix}_platform_joint" type="prismatic">
 			<origin xyz="0.0 0.0 0.285" rpy="0 0 0 " />
 			<parent link="${parent}"/>
-			<child link="${prefix}_elevator_link" />
+			<child link="${prefix}_platform_link" />
 			<axis xyz="0 0 1"/>
-			<limit effort="1.0" lower="0.0" upper="0.06" velocity="0.5"/>
+			<limit effort="1.0" lower="0.0" upper="0.05" velocity="0.5"/>
 	</joint>
-	<link name="${prefix}_elevator_link">
+	<link name="${prefix}_platform_link">
 		<visual>
 			<origin xyz="0 0 0" rpy="0 0 0" />

Commit message: description: setting elevator collision model as a box

File: rb2_description/urdf/elevator/elevator.urdf.xacro (robot description, xacro)
@@ -40,10 +40,10 @@
 		<collision>
 			<origin xyz="0 0 -0.0" rpy="0 0 0 " />
+			<geometry>
+				<box size="0.65 0.5 0.025" />
+			</geometry>
 			<!--geometry>
-				<box size="0.837 0.590 0.05" />
-			</geometry-->
-			<geometry>
 					<mesh filename="package://rb2_description/meshes/elevator/rb2_elevator.dae"/>
-				</geometry>
+				</geometry-->
 		</collision>
 		<inertial>
