Commit message: Added picking contact link to urdf

File: rb2_description/urdf/bases/rb2.urdf.xacro (robot description, xacro)
@@ -53,10 +53,18 @@
   <!-- DOCKING CONTACTS -->
   <joint name="${prefix}docking_joint" type="fixed">
-     <origin xyz="0.361 0.0 0.0" rpy="0 0 0" />
-     <parent link="${prefix}base_link"/>
-     <child link="${prefix}docking_contact_link" />
+    <origin xyz="0.361 0.0 0.0" rpy="0 0 0" />
+    <parent link="${prefix}base_link"/>
+    <child link="${prefix}docking_contact_link" />
   </joint>
   <!-- DOCKING LINK -->
   <link name="${prefix}docking_contact_link" />
+  <!-- PICKING CONTACTS -->
+  <joint name="${prefix}picking_joint" type="fixed">
+    <origin xyz="0.476 0.0 0.116" rpy="0 0 0" />
+    <parent link="${prefix}base_link"/>
+    <child link="${prefix}picking_contact_link" />
+  </joint>
+  <!-- PICKING LINK -->
+  <link name="${prefix}picking_contact_link" />
   </xacro:macro>
 </robot>

Commit message: rb2_description: added front and rear contacts

File: rb2_description/urdf/bases/rb2.urdf.xacro (robot description, xacro)
@@ -67,4 +67,20 @@
   <!-- PICKING LINK -->
   <link name="${prefix}picking_contact_link" />
+  <!-- FRONT CONTACTS -->
+  <joint name="${prefix}front_joint" type="fixed">
+    <origin xyz="0.476 0.0 0.116" rpy="0 0 0" />
+    <parent link="${prefix}base_link"/>
+    <child link="${prefix}front_contact_link" />
+  </joint>
+  <!-- FRONT LINK -->
+  <link name="${prefix}front_contact_link" />
+  <!-- REAR CONTACTS -->
+  <joint name="${prefix}rear_joint" type="fixed">
+    <origin xyz="-0.476 0.0 0.116" rpy="0 0 0" />
+    <parent link="${prefix}base_link"/>
+    <child link="${prefix}rear_contact_link" />
+  </joint>
+  <!-- REAR LINK -->
+  <link name="${prefix}rear_contact_link" />
   </xacro:macro>
 </robot>
