Commit message: Set new motors parameters

File: rb2_description/urdf/wheels/rubber_wheel.urdf.xacro (robot description, xacro)
@@ -5,5 +5,5 @@
 	<xacro:property name="M_PI" value="3.1415926535897931" />
 	<!-- Wheels -->
-	<xacro:property name="wheel_radius" value="0.110" />
+	<xacro:property name="wheel_radius" value="0.09" />
 	<xacro:property name="wheel_height" value="0.07" />
 	<xacro:property name="wheel_mass" value="0.3" /> <!-- in kg-->
